File: SimpleServoPS_PCB/SimpleServoCtrl.kicad_pcb (KiCad board)
At the start: 2 copper layers, 63.5 x 48.3 mm, 55 parts, among them J1 CONN_01X04, J2 Conn_01x08, J3 Conn_01x08, J4 Conn_01x08, J5 Conn_01x08, J6 Conn_01x08, J7 Conn_01x08, J8 Conn_01x05, P1 Conn_01x02, SW1 SW_Push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

Commit message: Rev A
Parts:
- D4: value DIODE -> D_Filled
- turned D1 to 0 degrees
- turned D2 to 0 degrees
- turned D3 to 0 degrees
- turned D4 to 180 degrees
Connections:
- D1 pad 1: Net-(D1-Pad1) -> SW1
- D1 pad 2: SW1 -> Net-(R17-Pad2)
- D2 pad 1: Net-(D2-Pad1) -> SW2
- D2 pad 2: SW2 -> Net-(R19-Pad2)
- D3 pad 1: Net-(D3-Pad1) -> SW3
- D3 pad 2: SW3 -> Net-(R21-Pad2)
- D4 pad 1: +12V -> Net-(C1-Pad1)
- D4 pad 2: Net-(C1-Pad1) -> +12V
- R17 pad 2: Net-(D1-Pad1) -> Net-(R17-Pad2)
- R18 pad 1: Net-(D1-Pad1) -> Net-(R17-Pad2)
- R19 pad 2: Net-(D2-Pad1) -> Net-(R19-Pad2)
- R20 pad 1: Net-(D2-Pad1) -> Net-(R19-Pad2)
- R21 pad 2: Net-(D3-Pad1) -> Net-(R21-Pad2)
- R22 pad 1: Net-(D3-Pad1) -> Net-(R21-Pad2)
Routing:
- net Net-(R21-Pad2): track 0.00 -> 4.55 mm
- net Net-(D3-Pad1): track 4.55 -> 0.00 mm
- net Net-(R17-Pad2): track 0.00 -> 4.55 mm
- net Net-(D1-Pad1): track 4.55 -> 0.00 mm
- net Net-(R19-Pad2): track 0.00 -> 4.55 mm
- net Net-(D2-Pad1): track 4.55 -> 0.00 mm
Other:
- board text added: "Simple Servo Controller 16 Packet Serial Version Rev. A DMFE 2021"
- board text removed: "Simple Servo Controller 16 Packet Serial Version Rev. n/c DMFE 2021"
