File: SimpleServoPS_PCB/SimpleServoCtrl.kicad_sch (KiCad schematic)
At the start: 51 parts, among them J1 CONN_01X04, J2 Conn_01x08, J3 Conn_01x08, J4 Conn_01x08, J5 Conn_01x08, J6 Conn_01x08, J7 Conn_01x08, J8 Conn_01x05, P1 Conn_01x02, SW1 SW_Push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

Commit message: Rev A
Parts:
- removed D1, D2, D3: LED, LED_SMD:LED_1206_3216Metric_Pad1.42x1.75mm_HandSolder, symbol SimpleServoCtrl-rescue:LED-RESCUE-SimpleServoCtrl
- removed D4: DIODE, Diode_SMD:D_SMA_Handsoldering, symbol SimpleServoCtrl-rescue:DIODE
- added D1, D2, D3: LED, symbol Device:LED_Filled
- added D4: D_Filled, symbol Device:D_Filled
Connections:
- net +12V: now also D4.2 (A)
- net SW1: now also D1.1 (K)
- net SW2: now also D2.1 (K)
- net SW3: now also D3.1 (K)
- net at R17.2, R18.1: now also D1.2 (A)
- net at R19.2, R20.1: now also D2.2 (A)
- net at R21.2, R22.1: now also D3.2 (A)
- net at C1.1, U4.3 (IN): now also D4.1 (K)
Other:
- note added: "Rev. A Diode pin numbers reversed"
Changed lines of the file:
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@@
     (title "Simple Servo Controller 16")
     (date "2021-03-12")
-    (rev "n/c")
+    (rev "A")
     (company "DMFE")
     (comment 1 "Packet Serial Version")
@@
     (stroke (width 0) (type solid) (color 0 0 0 0))
   )
-  (wire (pts (xy 48.26 25.4) (xy 49.53 25.4))
+  (wire (pts (xy 48.26 25.4) (xy 52.07 25.4))
     (stroke (width 0) (type solid) (color 0 0 0 0))
   )
@@
     (stroke (width 0) (type solid) (color 0 0 0 0))
   )
+  (wire (pts (xy 92.71 33.02) (xy 92.71 35.56))
+    (stroke (width 0) (type solid) (color 0 0 0 0))
+  )
   (wire (pts (xy 92.71 33.02) (xy 97.79 33.02))
     (stroke (width 0) (type solid) (color 0 0 0 0))
@@
     (stroke (width 0) (type solid) (color 0 0 0 0))
   )
+  (wire (pts (xy 104.14 33.02) (xy 104.14 35.56))
+    (stroke (width 0) (type solid) (color 0 0 0 0))
+  )
   (wire (pts (xy 104.14 33.02) (xy 109.22 33.02))
     (stroke (width 0) (type solid) (color 0 0 0 0))
@@
     (stroke (width 0) (type solid) (color 0 0 0 0))
   )
+  (wire (pts (xy 115.57 33.02) (xy 115.57 35.56))
+    (stroke (width 0) (type solid) (color 0 0 0 0))
+  )
   (wire (pts (xy 115.57 33.02) (xy 120.65 33.02))
     (stroke (width 0) (type solid) (color 0 0 0 0))
@@
   )
   (text "Vpp\nVdd\nVss\nPGD\nPGC" (at 25.4 149.86 180)
+    (effects (font (size 1.524 1.524)) (justify right bottom))
+  )
+  (text "Rev. A Diode pin numbers reversed" (at 57.15 198.12 180)
     (effects (font (size 1.524 1.524)) (justify right bottom))
   )
@@
     (pin "2")
   )
-  (symbol (lib_id "SimpleServoCtrl-rescue:DIODE") (at 54.61 25.4 0) (unit 1)
-    (in_bom yes) (on_board yes)
-    (property "Reference" "D4" (id 0) (at 54.61 22.86 0)
-      (effects (font (size 1.016 1.016)))
-    )
-    (property "Value" "DIODE" (id 1) (at 54.61 27.94 0)
-      (effects (font (size 1.016 1.016)) hide)
-    )
-    (property "Footprint" "Diode_SMD:D_SMA_Handsoldering" (id 2) (at 54.61 25.4 0)
-      (effects (font (size 1.524 1.524)) hide)
-    )
-    (property "Datasheet" "" (id 3) (at 54.61 25.4 0)
-      (effects (font (size 1.524 1.524)) hide)
-    )
-    (pin "1")
-    (pin "2")
-  )
-  (symbol (lib_id "SimpleServoCtrl-rescue:LED-RESCUE-SimpleServoCtrl") (at 92.71 38.1 270) (unit 1)
-    (in_bom yes) (on_board yes)
-    (property "Reference" "D1" (id 0) (at 95.25 38.1 0))
-    (property "Value" "LED" (id 1) (at 90.17 38.1 0))
-    (property "Footprint" "LED_SMD:LED_1206_3216Metric_Pad1.42x1.75mm_HandSolder" (id 2) (at 92.71 38.1 0)
-      (effects (font (size 1.524 1.524)) hide)
-    )
-    (property "Datasheet" "" (id 3) (at 92.71 38.1 0)
-      (effects (font (size 1.524 1.524)) hide)
-    )
-    (pin "1")
-    (pin "2")
-  )
-  (symbol (lib_id "SimpleServoCtrl-rescue:LED-RESCUE-SimpleServoCtrl") (at 104.14 38.1 270) (unit 1)
-    (in_bom yes) (on_board yes)
-    (property "Reference" "D2" (id 0) (at 106.68 38.1 0))
-    (property "Value" "LED" (id 1) (at 101.6 38.1 0))
-    (property "Footprint" "LED_SMD:LED_1206_3216Metric_Pad1.42x1.75mm_HandSolder" (id 2) (at 104.14 38.1 0)
-      (effects (font (size 1.524 1.524)) hide)
-    )
-    (property "Datasheet" "" (id 3) (at 104.14 38.1 0)
-      (effects (font (size 1.524 1.524)) hide)
-    )
-    (pin "1")
-    (pin "2")
-  )
-  (symbol (lib_id "SimpleServoCtrl-rescue:LED-RESCUE-SimpleServoCtrl") (at 115.57 38.1 270) (unit 1)
-    (in_bom yes) (on_board yes)
-    (property "Reference" "D3" (id 0) (at 118.11 38.1 0))
-    (property "Value" "LED" (id 1) (at 113.03 38.1 0))
-    (property "Footprint" "LED_SMD:LED_1206_3216Metric_Pad1.42x1.75mm_HandSolder" (id 2) (at 115.57 38.1 0)
-      (effects (font (size 1.524 1.524)) hide)
-    )
-    (property "Datasheet" "" (id 3) (at 115.57 38.1 0)
-      (effects (font (size 1.524 1.524)) hide)
+  (symbol (lib_id "Device:D_Filled") (at 55.88 25.4 0) (mirror y) (unit 1)
+    (in_bom yes) (on_board yes)
+    (property "Reference" "D4" (id 0) (at 55.88 21.59 0))
+    (property "Value" "D_Filled" (id 1) (at 55.88 21.59 0)
+      (effects (font (size 1.27 1.27)) hide)
+    )
+    (property "Footprint" "" (id 2) (at 55.88 25.4 0)
+      (effects (font (size 1.27 1.27)) hide)
+    )
+    (property "Datasheet" "~" (id 3) (at 55.88 25.4 0)
+      (effects (font (size 1.27 1.27)) hide)
+    )
+    (pin "1")
+    (pin "2")
+  )
+  (symbol (lib_id "Device:LED_Filled") (at 92.71 39.37 90) (unit 1)
+    (in_bom yes) (on_board yes)
+    (property "Reference" "D1" (id 0) (at 90.17 38.1 0)
+      (effects (font (size 1.27 1.27)) (justify right))
+    )
+    (property "Value" "LED" (id 1) (at 96.52 41.91 90)
+      (effects (font (size 1.27 1.27)) (justify right) hide)
+    )
+    (property "Footprint" "" (id 2) (at 92.71 39.37 0)
+      (effects (font (size 1.27 1.27)) hide)
+    )
+    (property "Datasheet" "~" (id 3) (at 92.71 39.37 0)
+      (effects (font (size 1.27 1.27)) hide)
+    )
+    (pin "1")
+    (pin "2")
+  )
+  (symbol (lib_id "Device:LED_Filled") (at 104.14 39.37 90) (unit 1)
+    (in_bom yes) (on_board yes)
+    (property "Reference" "D2" (id 0) (at 101.6 38.1 0)
+      (effects (font (size 1.27 1.27)) (justify right))
+    )
+    (property "Value" "LED" (id 1) (at 107.95 41.91 90)
+      (effects (font (size 1.27 1.27)) (justify right) hide)
+    )
+    (property "Footprint" "" (id 2) (at 104.14 39.37 0)
+      (effects (font (size 1.27 1.27)) hide)
+    )
+    (property "Datasheet" "~" (id 3) (at 104.14 39.37 0)
+      (effects (font (size 1.27 1.27)) hide)
+    )
+    (pin "1")
+    (pin "2")
+  )
+  (symbol (lib_id "Device:LED_Filled") (at 115.57 39.37 90) (unit 1)
+    (in_bom yes) (on_board yes)
+    (property "Reference" "D3" (id 0) (at 113.03 38.1 0)
+      (effects (font (size 1.27 1.27)) (justify right))
+    )
+    (property "Value" "LED" (id 1) (at 119.38 41.91 90)
+      (effects (font (size 1.27 1.27)) (justify right) hide)
+    )
+    (property "Footprint" "" (id 2) (at 115.57 39.37 0)
+      (effects (font (size 1.27 1.27)) hide)
+    )
+    (property "Datasheet" "~" (id 3) (at 115.57 39.37 0)
+      (effects (font (size 1.27 1.27)) hide)
     )
     (pin "1")
@@
       (reference "C9") (unit 1) (value "0.1uf") (footprint "Capacitor_SMD:C_0805_2012Metric_Pad1.18x1.45mm_HandSolder")
     )
-    (path "/00000000-0000-0000-0000-00005369c63d"
-      (reference "D1") (unit 1) (value "LED") (footprint "LED_SMD:LED_1206_3216Metric_Pad1.42x1.75mm_HandSolder")
-    )
-    (path "/00000000-0000-0000-0000-00005369c66d"
-      (reference "D2") (unit 1) (value "LED") (footprint "LED_SMD:LED_1206_3216Metric_Pad1.42x1.75mm_HandSolder")
-    )
-    (path "/00000000-0000-0000-0000-00005369c678"
-      (reference "D3") (unit 1) (value "LED") (footprint "LED_SMD:LED_1206_3216Metric_Pad1.42x1.75mm_HandSolder")
-    )
-    (path "/00000000-0000-0000-0000-00005369d6a9"
-      (reference "D4") (unit 1) (value "DIODE") (footprint "Diode_SMD:D_SMA_Handsoldering")
+    (path "/031f2283-76e4-4142-83e5-47878e0364ef"
+      (reference "D1") (unit 1) (value "LED") (footprint "")
+    )
+    (path "/a0766112-a833-4cc1-9e19-67f63404777a"
+      (reference "D2") (unit 1) (value "LED") (footprint "")
+    )
+    (path "/a8b59718-ab4a-4384-a54e-fcbe79e68c07"
+      (reference "D3") (unit 1) (value "LED") (footprint "")
+    )
+    (path "/6252cae2-7d72-4c29-be7a-9eed40323427"
+      (reference "D4") (unit 1) (value "D_Filled") (footprint "")
     )
     (path "/00000000-0000-0000-0000-000056e350fc"
